File: Hardware/NanoPage/NanoPage.kicad_pcb (KiCad board)
At the start: 6 copper layers, 91.8 x 37.5 mm, 93 parts, among them J1 TYPE-C-31-M-12, J2 Micro_SD_Card_Det, J3 FPC-05FB-24PH20, J4 BM03B-SRSS-TB, J5 SM02B-SRSS-TB_LF, J6 Conn_01x07, Q1 Si1308EDL, U1 USBLC6-2SC6, U2 TPS2116DRLR, U3 BQ25170DSGR, U4 MAX17055ETB+T, U5 PCF85063ATL, U6 TPS22929D, U7 TPS7A0233DBVR, U8 E73-2G4M08S1C, Y1 32.768kHz, Y2 32.768kHz

Commit message: fix: Update resistor value
Parts:
- J6: value Conn_01x07 -> ext_buttons_conn
- R5: value 100k -> 10k
Changed lines of the file:
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@@
 			)
 		)
-		(property "Value" "Conn_01x07"
+		(property "Value" "ext_buttons_conn"
 			(at 0 4.2 0)
 			(unlocked yes)
@@
 		(sheetname "/Buttons/")
 		(sheetfile "buttons.kicad_sch")
+		(units
+			(unit
+				(name "A")
+				(pins "1" "2" "3" "4" "5" "6" "7")
+			)
+		)
 		(attr smd)
 		(duplicate_pad_numbers_are_jumpers no)
@@
 			)
 		)
-		(attr smd)
+		(attr smd dnp)
 		(duplicate_pad_numbers_are_jumpers no)
 		(fp_line
@@
 			)
 		)
-		(property "Value" "100k"
+		(property "Value" "10k"
 			(at 0 1.17 0)
 			(layer "F.Fab")
@@
 			(keep_text_aligned yes)
 		)
-		(gr_text "3.5"
+		(gr_text "3,5"
 			(at 191.45 78.55 0)
 			(layer "Dwgs.User")
@@
 			(keep_text_aligned yes)
 		)
-		(gr_text "21.5"
+		(gr_text "21,5"
 			(at 205.75 104.25 90)
 			(layer "Dwgs.User")
@@
 			(keep_text_aligned yes)
 		)
-		(gr_text "37.5"
+		(gr_text "37,5"
 			(at 90.15 104.25 90)
 			(layer "Dwgs.User")
@@
 			(keep_text_aligned yes)
 		)
-		(gr_text "91.8"
+		(gr_text "91,8"
 			(at 147.29997 73.7976 0)
 			(layer "Dwgs.User")

Commit message: fix: bump R5 (USB_DETECT) pull-up to 931k, cutting a confirmed 330uA leak
Direct multimeter ammeter measurement (not the fuel gauge) put the
true idle draw at 880uA on a battery without a protection circuit,
confirming R5's TPS2116 ST pull-up as a real, continuous ~330uA path.
Reworked 10k -> 931k in the same 0402 footprint (drop-in bench
rework), checked safe against the TPS2116's leakage/VOL/response-time
specs - expected new draw ~3.5uA, not yet re-verified on hardware.

Also records this session's fuel-gauge-vs-multimeter comparison
(AvgCurrent tracks closely; raw Current reads 5-24% high and noisier -
R11's tolerance and the multimeter's own accuracy spec were both
checked and ruled out as the cause), and why R8/R9/R12/R14 - the same
open-drain-status-pin class as R5 - were evaluated but deliberately
left at 10k this round: their chips' higher leakage specs rule out
reusing 931k for them, R8/R9 only matter while USB is already
supplying far more current than that, and R12/R14 are an accepted
latent-risk bet rather than a current cost.
Parts:
- R5: value 10k -> 931k
Changed lines of the file:
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@@
 			)
 		)
-		(property "Value" "10k"
+		(property "Value" "931k"
 			(at 0 1.17 0)
 			(layer "F.Fab")
