File: Hardware/NanoPage/NanoPage.kicad_pcb (KiCad board)
At the start: 6 copper layers, 91.8 x 37.5 mm, 93 parts, among them J1 TYPE-C-31-M-12, J2 Micro_SD_Card_Det, J3 FPC-05FB-24PH20, J4 BM03B-SRSS-TB, J5 SM02B-SRSS-TB_LF, J6 ext_buttons_conn, Q1 Si1308EDL, U1 USBLC6-2SC6, U2 TPS2116DRLR, U3 BQ25170DSGR, U4 MAX17055ETB+T, U5 PCF85063ATL, U6 TPS22929D, U7 TPS7A0233DBVR, U8 E73-2G4M08S1C, Y1 32.768kHz, Y2 32.768kHz

Commit message: feat: vendor custom KiCad symbols, footprints and 3D models into the project
Move all downloaded and self-made parts into a project-local NanoPage
library (libraries/NanoPage.{kicad_sym,pretty,3dshapes}) referenced via
${KIPRJMOD}, so the design opens on any machine without the global
external_libraries folder. KiCad built-in parts are unchanged.
Parts:
- FL1: footprint Personal Library:L_CommonModeChoke_TDK_0503USB -> NanoPage:L_CommonModeChoke_TDK_0503USB
- J1: footprint TYPE-C-31-M-12:HRO_TYPE-C-31-M-12 -> NanoPage:HRO_TYPE-C-31-M-12
- J3: footprint Personal Library:XUNPU FPC-05FB-24PH20 -> NanoPage:XUNPU FPC-05FB-24PH20
- J4: footprint BM03B-SRSS-TB:BM03BSRSSTBLFSN -> NanoPage:BM03BSRSSTBLFSN
- J5: footprint SM02B-SRSS-TB:SM02BSRSSTBLFSN -> NanoPage:SM02BSRSSTBLFSN
- J6: footprint Personal Library:HC-FPC-05-09-5RLTAG -> NanoPage:HC-FPC-05-09-5RLTAG
- L1: footprint Personal Library:NR4018 -> NanoPage:NR4018
- S1, S2, S3: footprint SKRTLAE010:SKRTLAE010 -> NanoPage:SKRTLAE010
- S4: footprint PTS526SM15SMTR2:PTS526SM15SMTR2LFS -> NanoPage:PTS526SM15SMTR2LFS
- U2: footprint TPS2116DRL:SOTFL50P160X60-8N -> NanoPage:SOTFL50P160X60-8N
- U3: footprint Personal Library:BQ25170 -> NanoPage:BQ25170
- U4: footprint MAX17055ETB-T:SON40P250X200X80-11N -> NanoPage:SON40P250X200X80-11N
- U5: footprint PCF85063ATL:SON50P260X260X50-11N -> NanoPage:SON50P260X260X50-11N
- U8: footprint E73-2G4M08S1C:E73-2G4M08S1C -> NanoPage:E73-2G4M08S1C
Changed lines of the file:
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@@
 		)
 	)
-	(footprint "Personal Library:L_CommonModeChoke_TDK_0503USB"
+	(footprint "NanoPage:L_CommonModeChoke_TDK_0503USB"
 		(layer "F.Cu")
 		(at 146.85 102.95)
@@
 		)
 	)
-	(footprint "SKRTLAE010:SKRTLAE010"
+	(footprint "NanoPage:SKRTLAE010"
 		(locked yes)
 		(layer "F.Cu")
@@
 		)
 		(embedded_fonts no)
-		(model "SKRTLAE010.stp"
+		(model "${KIPRJMOD}/libraries/NanoPage.3dshapes/SKRTLAE010.step"
 			(offset
 				(xyz 0.03 -0.5 1.73)
@@
 		)
 	)
-	(footprint "E73-2G4M08S1C:E73-2G4M08S1C"
+	(footprint "NanoPage:E73-2G4M08S1C"
 		(locked yes)
 		(layer "F.Cu")
@@
 		)
 		(embedded_fonts no)
-		(model "/home/vagarth/Applications/Kicad/external_libraries/E73-2G4M08S1C/E73-2G4M08S1C.step"
+		(model "${KIPRJMOD}/libraries/NanoPage.3dshapes/E73-2G4M08S1C.step"
 			(offset
 				(xyz 0 0 0)
@@
 		)
 		(embedded_fonts no)
-		(model "/home/vagarth/Applications/Kicad/external_libraries/3D models/104031-0811.STEP"
+		(model "${KIPRJMOD}/libraries/NanoPage.3dshapes/104031-0811.step"
 			(offset
 				(xyz 0 0 0)
@@
 		)
 	)
-	(footprint "PCF85063ATL:SON50P260X260X50-11N"
+	(footprint "NanoPage:SON50P260X260X50-11N"
 		(layer "F.Cu")
 		(at 114.25 117.5 180)
@@
 		)
 		(embedded_fonts no)
-		(model "/home/vagarth/Applications/Kicad/external_libraries/PCF85063ATL/PCF85063ATL.stp"
+		(model "${KIPRJMOD}/libraries/NanoPage.3dshapes/PCF85063ATL.step"
 			(offset
 				(xyz 0 0 0)
@@
 		)
 	)
-	(footprint "Personal Library:HC-FPC-05-09-5RLTAG"
+	(footprint "NanoPage:HC-FPC-05-09-5RLTAG"
 		(layer "F.Cu")
 		(at 125.4 119.675)
@@
 		)
 	)
-	(footprint "Personal Library:XUNPU FPC-05FB-24PH20"
+	(footprint "NanoPage:XUNPU FPC-05FB-24PH20"
 		(locked yes)
 		(layer "F.Cu")
@@
 		)
 		(embedded_fonts no)
-		(model "/home/vagarth/Applications/Kicad/external_libraries/3D models/FPC-05FB-24PH20.STEP"
+		(model "${KIPRJMOD}/libraries/NanoPage.3dshapes/FPC-05FB-24PH20.step"
 			(offset
 				(xyz 0 -3.5 0)
@@
 		)
 	)
-	(footprint "SM02B-SRSS-TB:SM02BSRSSTBLFSN"
+	(footprint "NanoPage:SM02BSRSSTBLFSN"
 		(layer "F.Cu")
 		(at 168.188 92.2 90)
@@
 		)
 		(embedded_fonts no)
-		(model "/home/vagarth/Applications/Kicad/external_libraries/3D models/SM02B-SRSS-TB (LF)(SN).STEP"
+		(model "${KIPRJMOD}/libraries/NanoPage.3dshapes/SM02B-SRSS-TB.step"
 			(offset
 				(xyz 0 0 0)
@@
 		)
 	)
-	(footprint "MAX17055ETB-T:SON40P250X200X80-11N"
+	(footprint "NanoPage:SON40P250X200X80-11N"
 		(layer "F.Cu")
 		(at 157.56 91.56 90)
@@
 		)
 		(embedded_fonts no)
-		(model "MAX17055ETB+T.stp"
+		(model "${KIPRJMOD}/libraries/NanoPage.3dshapes/MAX17055ETB.step"
 			(offset
 				(xyz 0 0 0)
@@
 		)
 	)
-	(footprint "BM03B-SRSS-TB:BM03BSRSSTBLFSN"
+	(footprint "NanoPage:BM03BSRSSTBLFSN"
 		(layer "F.Cu")
 		(at 134.1 90.713 180)
@@
 		)
 		(embedded_fonts no)
-		(model "/home/vagarth/Applications/Kicad/external_libraries/BM03B-SRSS-TB_LF_SN/BM03B-SRSS-TB-LF__SN.STEP"
+		(model "${KIPRJMOD}/libraries/NanoPage.3dshapes/BM03B-SRSS-TB.step"
 			(offset
 				(xyz 0 0 0)
@@
 		)
 	)
-	(footprint "Personal Library:NR4018"
+	(footprint "NanoPage:NR4018"
 		(layer "F.Cu")
 		(at 167.75 110.75 -90)
@@
 		)
 		(embedded_fonts no)
-		(model "/home/vagarth/Applications/Kicad/external_libraries/3D models/NR4018.step"
+		(model "${KIPRJMOD}/libraries/NanoPage.3dshapes/NR4018.step"
 			(offset
 				(xyz 0 0 0)
@@
 		)
 	)
-	(footprint "TPS2116DRL:SOTFL50P160X60-8N"
+	(footprint "NanoPage:SOTFL50P160X60-8N"
 		(layer "F.Cu")
 		(at 160.6 99.1)
@@
 		)
 		(embedded_fonts no)
-		(model "/home/vagarth/Applications/Kicad/external_libraries/TPS2116DRLR/TPS2116DRLR.step"
+		(model "${KIPRJMOD}/libraries/NanoPage.3dshapes/TPS2116DRLR.step"
 			(offset
 				(xyz 0 0 0)
@@
 		(embedded_fonts no)
 	)
-	(footprint "PTS526SM15SMTR2:PTS526SM15SMTR2LFS"
+	(footprint "NanoPage:PTS526SM15SMTR2LFS"
 		(layer "F.Cu")
 		(at 132.1 102.5)
@@
 		)
 		(embedded_fonts no)
-		(model "/home/vagarth/Applications/Kicad/external_libraries/PTS526SM15SMTR2_LFS/PTS526SM15SMTR2_LFS.stp"
+		(model "${KIPRJMOD}/libraries/NanoPage.3dshapes/PTS526SM15SMTR2.step"
 			(offset
 				(xyz 0 0 0.04999999999)
@@
 		)
 	)
-	(footprint "SKRTLAE010:SKRTLAE010"
+	(footprint "NanoPage:SKRTLAE010"
 		(locked yes)
 		(layer "F.Cu")
@@
 		)
 		(embedded_fonts no)
-		(model "SKRTLAE010.stp"
+		(model "${KIPRJMOD}/libraries/NanoPage.3dshapes/SKRTLAE010.step"
 			(offset
 				(xyz 0.03 -0.5 1.73)
@@
 		)
 	)
-	(footprint "TYPE-C-31-M-12:HRO_TYPE-C-31-M-12"
+	(footprint "NanoPage:HRO_TYPE-C-31-M-12"
 		(locked yes)
 		(layer "F.Cu")
@@
 		)
 		(embedded_fonts no)
-		(model "/home/vagarth/Applications/Kicad/external_libraries/TYPE-C-31-M-12/TYPE-C-31-M-12.step"
+		(model "${KIPRJMOD}/libraries/NanoPage.3dshapes/TYPE-C-31-M-12.step"
 			(offset
 				(xyz 0 0 0)
@@
 		)
 	)
-	(footprint "SKRTLAE010:SKRTLAE010"
+	(footprint "NanoPage:SKRTLAE010"
 		(locked yes)
 		(layer "F.Cu")
@@
 		)
 		(embedded_fonts no)
-		(model "SKRTLAE010.stp"
+		(model "${KIPRJMOD}/libraries/NanoPage.3dshapes/SKRTLAE010.step"
 			(offset
 				(xyz 0.03 -0.5 1.73)
@@
 		)
 	)
-	(footprint "Personal Library:BQ25170"
+	(footprint "NanoPage:BQ25170"
 		(layer "F.Cu")
 		(at 167.95 102.05)
