File: Hardware/NanoPage/battery_charger_and_fuel_guage.kicad_sch (KiCad schematic)
At the start: 14 parts, among them J5 SM02B-SRSS-TB_LF, U3 BQ25170DSGR, U4 MAX17055ETB+T

Commit message: fix: Fix wrong footprint
Parts:
- J5: footprint SM02B-SRSS-TB(LF)(SN):SM02BSRSSTBLFSN -> SM02B-SRSS-TB:SM02BSRSSTBLFSN
- U3: footprint Personal library:BQ25170 -> Personal Library:BQ25170
- U4: footprint MAX17055ETB+T:SON40P250X200X80-11N -> MAX17055ETB-T:SON40P250X200X80-11N
Changed lines of the file:
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@@
 			)
 		)
-		(property "Footprint" "Personal library:BQ25170"
+		(property "Footprint" "Personal Library:BQ25170"
 			(at 64.77 100.33 0)
 			(hide yes)
@@
 			)
 		)
-		(property "Footprint" "SM02B-SRSS-TB(LF)(SN):SM02BSRSSTBLFSN"
+		(property "Footprint" "SM02B-SRSS-TB:SM02BSRSSTBLFSN"
 			(at 251.46 192.71 0)
 			(hide yes)
@@
 			)
 		)
-		(property "Footprint" "MAX17055ETB+T:SON40P250X200X80-11N"
+		(property "Footprint" "MAX17055ETB-T:SON40P250X200X80-11N"
 			(at 175.26 182.55 0)
 			(hide yes)

Commit message: feat: vendor custom KiCad symbols, footprints and 3D models into the project
Move all downloaded and self-made parts into a project-local NanoPage
library (libraries/NanoPage.{kicad_sym,pretty,3dshapes}) referenced via
${KIPRJMOD}, so the design opens on any machine without the global
external_libraries folder. KiCad built-in parts are unchanged.
Parts:
- J5: footprint SM02B-SRSS-TB:SM02BSRSSTBLFSN -> NanoPage:SM02BSRSSTBLFSN; symbol SM02B-SRSS-TB(LF)(SN):SM02B-SRSS-TB_LF__SN_ -> NanoPage:SM02B-SRSS-TB_LF__SN_
- U3: footprint Personal Library:BQ25170 -> NanoPage:BQ25170; symbol personal-library:BQ25170DSGR -> NanoPage:BQ25170DSGR
- U4: footprint MAX17055ETB-T:SON40P250X200X80-11N -> NanoPage:SON40P250X200X80-11N; symbol MAX17055ETB+T:MAX17055ETB+T -> NanoPage:MAX17055ETB+T
Changed lines of the file:
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@@
 	)
 	(symbol
-		(lib_id "personal-library:BQ25170DSGR")
+		(lib_id "NanoPage:BQ25170DSGR")
 		(at 64.77 100.33 0)
 		(unit 1)
@@
 			)
 		)
-		(property "Footprint" "Personal Library:BQ25170"
+		(property "Footprint" "NanoPage:BQ25170"
 			(at 64.77 100.33 0)
 			(hide yes)
@@
 	)
 	(symbol
-		(lib_id "SM02B-SRSS-TB(LF)(SN):SM02B-SRSS-TB_LF__SN_")
+		(lib_id "NanoPage:SM02B-SRSS-TB_LF__SN_")
 		(at 232.41 97.79 0)
 		(unit 1)
@@
 			)
 		)
-		(property "Footprint" "SM02B-SRSS-TB:SM02BSRSSTBLFSN"
+		(property "Footprint" "NanoPage:SM02BSRSSTBLFSN"
 			(at 251.46 192.71 0)
 			(hide yes)
@@
 	)
 	(symbol
-		(lib_id "MAX17055ETB+T:MAX17055ETB+T")
+		(lib_id "NanoPage:MAX17055ETB+T")
 		(at 148.59 87.63 0)
 		(unit 1)
@@
 			)
 		)
-		(property "Footprint" "MAX17055ETB-T:SON40P250X200X80-11N"
+		(property "Footprint" "NanoPage:SON40P250X200X80-11N"
 			(at 175.26 182.55 0)
 			(hide yes)
