File: Hardware/NanoPage/display.kicad_sch (KiCad schematic)
At the start: 18 parts, among them J3 FPC-05FB-24PH20, Q1 Si1308EDL

Commit message: fix: Fix wrong footprint
Parts:
- J3: footprint Personal library:XUNPU FPC-05FB-24PH20 -> Personal Library:XUNPU FPC-05FB-24PH20
- L1: footprint Personal library:NR4018 -> Personal Library:NR4018
Changed lines of the file:
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@@
 			)
 		)
-		(property "Footprint" "Personal library:NR4018"
+		(property "Footprint" "Personal Library:NR4018"
 			(at 91.44 96.52 0)
 			(hide yes)
@@
 			)
 		)
-		(property "Footprint" "Personal library:XUNPU FPC-05FB-24PH20"
+		(property "Footprint" "Personal Library:XUNPU FPC-05FB-24PH20"
 			(at 222.25 101.6 0)
 			(hide yes)

Commit message: feat: vendor custom KiCad symbols, footprints and 3D models into the project
Move all downloaded and self-made parts into a project-local NanoPage
library (libraries/NanoPage.{kicad_sym,pretty,3dshapes}) referenced via
${KIPRJMOD}, so the design opens on any machine without the global
external_libraries folder. KiCad built-in parts are unchanged.
Parts:
- J3: footprint Personal Library:XUNPU FPC-05FB-24PH20 -> NanoPage:XUNPU FPC-05FB-24PH20
- L1: footprint Personal Library:NR4018 -> NanoPage:NR4018
Changed lines of the file:
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@@
 			)
 		)
-		(property "Footprint" "Personal Library:NR4018"
+		(property "Footprint" "NanoPage:NR4018"
 			(at 91.44 96.52 0)
 			(hide yes)
@@
 			)
 		)
-		(property "Footprint" "Personal Library:XUNPU FPC-05FB-24PH20"
+		(property "Footprint" "NanoPage:XUNPU FPC-05FB-24PH20"
 			(at 222.25 101.6 0)
 			(hide yes)
