File: Hardware/NanoPage/mcu.kicad_sch (KiCad schematic)
At the start: 15 parts, among them J4 BM03B-SRSS-TB, U8 E73-2G4M08S1C, Y2 32.768kHz

Commit message: fix: Fix wrong footprint
Parts:
- removed U8: E73-2G4M08S1C, Personal library:E73-2G4M08S1C, symbol personal-library:E73-2G4M08S1C-52840
- added U8: E73-2G4M08S1C, E73-2G4M08S1C:E73-2G4M08S1C, symbol Personal Library:E73-2G4M08S1C-52840
- J4: footprint BM03B-SRSS-TB(LF)(SN):BM03BSRSSTBLFSN -> BM03B-SRSS-TB:BM03BSRSSTBLFSN
Connections:
- net +3V3: now also U8.19 (VDD), U8.23 (VDDH)
- net DCCH: now also U8.25 (DCCH)
- net GND: now also U8.21 (GND), U8.24 (GND), U8.5 (GND)
- net MCU_ACTION_BTN: now also U8.41 (P0.09/NFC1)
- net MCU_ALERT: now also U8.33 (P0.13)
- net MCU_D+: now also U8.31 (USB_D+)
- net MCU_D-: now also U8.29 (USB_D-)
- net MCU_EPD_BUSY: now also U8.16 (P0.08)
- net MCU_EPD_CS: now also U8.12 (P0.26)
- net MCU_EPD_DC: now also U8.14 (P0.06)
- net MCU_EPD_RES: now also U8.15 (P0.05/AIN3)
- net MCU_NEXT_BTN: now also U8.43 (P0.10/NFC2)
- net MCU_PG: now also U8.36 (P1.00)
- net MCU_PREV_BTN: now also U8.35 (P0.24)
- net MCU_RESET: now also U8.26 (P0.18/RESET)
- net MCU_RTC_INT: now also U8.7 (P0.02/AIN0)
- net MCU_SD_CS: now also U8.17 (P1.09)
- net MCU_SD_DET: now also U8.20 (P0.12)
- net MCU_SD_ON: now also U8.1 (P1.11)
- net MCU_STAT: now also U8.3 (P0.03/AIN1)
- net MCU_SWCLK: now also U8.39 (SWDCLK)
- net MCU_SWDIO: now also U8.37 (SWDIO)
- net MCU_USB_DETECT: now also U8.30 (P0.17)
- net MISO: now also U8.8 (P0.29/AIN5)
- net MOSI: now also U8.10 (P0.30/AIN6)
- net SCL: now also U8.4 (P0.28/AIN4)
- net SCLK: now also U8.9 (P0.31/AIN7)
- net SDA: now also U8.6 (P1.13)
- net VBUS: now also U8.27 (VBUS)
- net XL1: now also U8.11 (P0.00/XL1)
- net XL2: now also U8.13 (P0.01/XL2)

Commit message: feat: vendor custom KiCad symbols, footprints and 3D models into the project
Move all downloaded and self-made parts into a project-local NanoPage
library (libraries/NanoPage.{kicad_sym,pretty,3dshapes}) referenced via
${KIPRJMOD}, so the design opens on any machine without the global
external_libraries folder. KiCad built-in parts are unchanged.
Parts:
- J4: footprint BM03B-SRSS-TB:BM03BSRSSTBLFSN -> NanoPage:BM03BSRSSTBLFSN; symbol BM03B-SRSS-TB(LF)(SN):BM03B-SRSS-TB_LF__SN_ -> NanoPage:BM03B-SRSS-TB_LF__SN_
- U8: footprint E73-2G4M08S1C:E73-2G4M08S1C -> NanoPage:E73-2G4M08S1C; symbol Personal Library:E73-2G4M08S1C-52840 -> NanoPage:E73-2G4M08S1C-52840
Changed lines of the file:
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@@
 	)
 	(symbol
-		(lib_id "BM03B-SRSS-TB(LF)(SN):BM03B-SRSS-TB_LF__SN_")
+		(lib_id "NanoPage:BM03B-SRSS-TB_LF__SN_")
 		(at 246.38 55.88 0)
 		(mirror y)
@@
 			)
 		)
-		(property "Footprint" "BM03B-SRSS-TB:BM03BSRSSTBLFSN"
+		(property "Footprint" "NanoPage:BM03BSRSSTBLFSN"
 			(at 227.33 150.8 0)
 			(hide yes)
@@
 	)
 	(symbol
-		(lib_id "Personal Library:E73-2G4M08S1C-52840")
+		(lib_id "NanoPage:E73-2G4M08S1C-52840")
 		(at 110.49 81.28 0)
 		(unit 1)
@@
 			)
 		)
-		(property "Footprint" "E73-2G4M08S1C:E73-2G4M08S1C"
+		(property "Footprint" "NanoPage:E73-2G4M08S1C"
 			(at 111.506 122.428 0)
 			(hide yes)
