File: Hardware/NanoPage/power.kicad_sch (KiCad schematic)
At the start: 18 parts, among them J1 TYPE-C-31-M-12, U1 USBLC6-2SC6, U2 TPS2116DRLR, U7 TPS7A0233DBVR

Commit message: fix: Fix wrong footprint
Parts:
- FL1: footprint Personal library:L_CommonModeChoke_TDK_0503USB -> Personal Library:L_CommonModeChoke_TDK_0503USB
- U2: footprint TPS2116:SOTFL50P160X60-8N -> TPS2116DRL:SOTFL50P160X60-8N
Changed lines of the file:
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@@
 			)
 		)
-		(property "Footprint" "TPS2116:SOTFL50P160X60-8N"
+		(property "Footprint" "TPS2116DRL:SOTFL50P160X60-8N"
 			(at 121.92 52.07 0)
 			(hide yes)
@@
 			)
 		)
-		(property "Footprint" "Personal library:L_CommonModeChoke_TDK_0503USB"
+		(property "Footprint" "Personal Library:L_CommonModeChoke_TDK_0503USB"
 			(at 170.18 156.21 0)
 			(hide yes)

Commit message: fix: Update resistor value
Parts:
- R5: value 100k -> 10k
Changed lines of the file:
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@@
 			)
 		)
-		(property "Value" "100k"
+		(property "Value" "10k"
 			(at 147.32 58.166 0)
 			(show_name no)

Commit message: fix: bump R5 (USB_DETECT) pull-up to 931k, cutting a confirmed 330uA leak
Direct multimeter ammeter measurement (not the fuel gauge) put the
true idle draw at 880uA on a battery without a protection circuit,
confirming R5's TPS2116 ST pull-up as a real, continuous ~330uA path.
Reworked 10k -> 931k in the same 0402 footprint (drop-in bench
rework), checked safe against the TPS2116's leakage/VOL/response-time
specs - expected new draw ~3.5uA, not yet re-verified on hardware.

Also records this session's fuel-gauge-vs-multimeter comparison
(AvgCurrent tracks closely; raw Current reads 5-24% high and noisier -
R11's tolerance and the multimeter's own accuracy spec were both
checked and ruled out as the cause), and why R8/R9/R12/R14 - the same
open-drain-status-pin class as R5 - were evaluated but deliberately
left at 10k this round: their chips' higher leakage specs rule out
reusing 931k for them, R8/R9 only matter while USB is already
supplying far more current than that, and R12/R14 are an accepted
latent-risk bet rather than a current cost.
Parts:
- R5: value 10k -> 931k
Changed lines of the file:
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@@
 			)
 		)
-		(property "Value" "10k"
+		(property "Value" "931k"
 			(at 147.32 58.166 0)
 			(show_name no)

Commit message: feat: vendor custom KiCad symbols, footprints and 3D models into the project
Move all downloaded and self-made parts into a project-local NanoPage
library (libraries/NanoPage.{kicad_sym,pretty,3dshapes}) referenced via
${KIPRJMOD}, so the design opens on any machine without the global
external_libraries folder. KiCad built-in parts are unchanged.
Parts:
- FL1: footprint Personal Library:L_CommonModeChoke_TDK_0503USB -> NanoPage:L_CommonModeChoke_TDK_0503USB
- J1: footprint TYPE-C-31-M-12:HRO_TYPE-C-31-M-12 -> NanoPage:HRO_TYPE-C-31-M-12; symbol TYPE-C-31-M-12:TYPE-C-31-M-12 -> NanoPage:TYPE-C-31-M-12
- U2: footprint TPS2116DRL:SOTFL50P160X60-8N -> NanoPage:SOTFL50P160X60-8N; symbol TPS2116:TPS2116DRLR -> NanoPage:TPS2116DRLR
- U7: symbol personal-library:TPS7A02 -> NanoPage:TPS7A02
Changed lines of the file:
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@@
 	)
 	(symbol
-		(lib_id "TPS2116:TPS2116DRLR")
+		(lib_id "NanoPage:TPS2116DRLR")
 		(at 121.92 52.07 0)
 		(unit 1)
@@
 			)
 		)
-		(property "Footprint" "TPS2116DRL:SOTFL50P160X60-8N"
+		(property "Footprint" "NanoPage:SOTFL50P160X60-8N"
 			(at 121.92 52.07 0)
 			(hide yes)
@@
 	)
 	(symbol
-		(lib_id "personal-library:TPS7A02")
+		(lib_id "NanoPage:TPS7A02")
 		(at 181.61 45.72 0)
 		(unit 1)
@@
 			)
 		)
-		(property "Footprint" "Personal Library:L_CommonModeChoke_TDK_0503USB"
+		(property "Footprint" "NanoPage:L_CommonModeChoke_TDK_0503USB"
 			(at 170.18 156.21 0)
 			(hide yes)
@@
 	)
 	(symbol
-		(lib_id "TYPE-C-31-M-12:TYPE-C-31-M-12")
+		(lib_id "NanoPage:TYPE-C-31-M-12")
 		(at 100.33 132.08 0)
 		(unit 1)
@@
 			)
 		)
-		(property "Footprint" "TYPE-C-31-M-12:HRO_TYPE-C-31-M-12"
+		(property "Footprint" "NanoPage:HRO_TYPE-C-31-M-12"
 			(at 100.33 132.08 0)
 			(hide yes)
