File: Hardware/NanoPage/rtc.kicad_sch (KiCad schematic)
At the start: 7 parts, among them U5 PCF85063ATL, Y1 32.768kHz

Commit message: feat: vendor custom KiCad symbols, footprints and 3D models into the project
Move all downloaded and self-made parts into a project-local NanoPage
library (libraries/NanoPage.{kicad_sym,pretty,3dshapes}) referenced via
${KIPRJMOD}, so the design opens on any machine without the global
external_libraries folder. KiCad built-in parts are unchanged.
Parts:
- U5: footprint PCF85063ATL:SON50P260X260X50-11N -> NanoPage:SON50P260X260X50-11N; symbol PCF85063ATL:PCF85063ATL_1,118 -> NanoPage:PCF85063ATL_1,118
Changed lines of the file:
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@@
 	)
 	(symbol
-		(lib_id "PCF85063ATL:PCF85063ATL_1,118")
+		(lib_id "NanoPage:PCF85063ATL_1,118")
 		(at 133.35 88.9 0)
 		(unit 1)
@@
 			)
 		)
-		(property "Footprint" "PCF85063ATL:SON50P260X260X50-11N"
+		(property "Footprint" "NanoPage:SON50P260X260X50-11N"
 			(at 165.1 183.82 0)
 			(hide yes)
